File: kicad/desk.kicad_sch (KiCad schematic)
At the start: 12 parts, among them J1 DIN harness, J2 ESP32 DevKit V1, J3 ESP32 DevKit V1, U1 PC817, U2 PC817

Commit message: Fix missing schematic<->board linkage; retire the PCB generator
Generated footprints carried no (path "/<symbol-uuid>"), so Update PCB
from Schematic could not match them and treated every symbol as new.
link_pcb.py injects the paths by reference designator. Board layout is
now hand-maintained; gen_pcb.py removed.

Co-Authored-By: Claude Opus 5 <noreply@anthropic.com>
Parts:
- R1, R2, R3, R4, R5, R6, R7: footprint Resistor_THT:R_Axial_DIN0207_L6.3mm_D2.5mm_P10.16mm_Horizontal -> Resistor_THT:R_Axial_DIN0207_L6.3mm_D2.5mm_P7.62mm_Horizontal
Connections:
- net GPIO16: no longer R5.2, R6.1
- net WHITE_UP: no longer R3.1
- net YELLOW_DN: no longer R4.1
- new net: R5.2, R6.1

Commit message: Board ready to cut: J4 pass-through, GND pour, 3 mounting holes, DRC clean
Export script matches the shop guide section 4 (4.6 gerbers, X2 and netlist
attrs off, merged inch Excellon) and now emits F.Silkscreen for the laser.
Footer corrected to solve-offsets: MX/MY are per-board, and this board is
not near page origin so the geo-aux-heat constants would run it off the
fixture entirely.

Co-Authored-By: Claude Opus 5 <noreply@anthropic.com>
Parts:
- added J4: DIN harness, TerminalBlock_Phoenix:TerminalBlock_Phoenix_MKDS-1,5-7_1x07_P5.00mm_Horizontal, symbol Connector_Generic:Conn_01x07
- added TP1: TestPoint_Square, TestPoint:TestPoint_Pad_2.0x2.0mm, symbol Connector:TestPoint_Square
Connections:
- net +5V: now also J4.2 (Pin_2)
- net BLACK_DATA: now also J4.5 (Pin_5)
- net GND: now also J4.1 (Pin_1), TP1.1
- net GPIO16: now also R5.2, R6.1
- net WHITE_UP: now also R3.1, J4.3 (Pin_3)
- net YELLOW_DN: now also R4.1, J4.4 (Pin_4)
- net HS3_GRN: now reaches J1.6 (Pin_6)
- net HS3_GRN: now also J4.6 (Pin_6)
- net HS4_BLUE: now reaches J1.7 (Pin_7)
- net HS4_BLUE: now also J4.7 (Pin_7)
- no-connect marks 27 -> 25
